File: schematicSheet/sensors.kicad_sch (KiCad schematic)
At the start: 18 parts, among them U10 MMC5983MA, U2 ADXL375BCCZ-RL7, U4 MS5607-02BA, U6 BMI088, U8 TMP275AIDGKR VSSOP8

Commit message: Arranged pin
Other:
- note removed: "C50 - C69"
Changed lines of the file:
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@@
-		)
-	)
-	(text "C50 - C69\n"
-		(exclude_from_sim no)
-		(at 26.162 19.812 0)
-		(effects
-			(font
-				(size 1.27 1.27)
-			)
 		)
 	)

Commit message: update label
Changed lines of the file:
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@@
 		)
 	)
-	(global_label "ACC_MISO"
+	(global_label "SPI_MISO"
 		(shape output)
 		(at 139.7 82.55 90)
@@
 		)
 		(property "Intersheetrefs" "${INTERSHEET_REFS}"
-			(at 139.7 74.0259 90)
+			(at 139.7 74.4069 90)
 			(effects
 				(font
@@
 		)
 	)
-	(global_label "ACC_SCLK"
+	(global_label "SPI_SCLK"
 		(shape input)
 		(at 134.62 82.55 90)
@@
 		)
 		(property "Intersheetrefs" "${INTERSHEET_REFS}"
-			(at 134.62 73.8988 90)
+			(at 134.62 74.2798 90)
 			(effects
 				(font
@@
 		)
 	)
-	(global_label "ACC_MOSI"
+	(global_label "SPI_MOSI"
 		(shape input)
 		(at 144.78 82.55 90)
@@
 		)
 		(property "Intersheetrefs" "${INTERSHEET_REFS}"
-			(at 144.78 74.0259 90)
-			(effects
-				(font
+			(at 144.78 74.4069 90)
+			(effects
+				(font

Commit message: update
Parts:
- R10, R11: value 2.2k -> 2.7k
Connections:
- net +3.3V: no longer C34.2, U10.2 (VDD)
- net GND: now also U2.2 (GND), U2.5 (GND)
- new net: C34.2, U10.2 (VDD)
Changed lines of the file:
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@@
 	)
 	(junction
-		(at 176.53 40.64)
-		(diameter 0)
-		(color 0 0 0 0)
-	)
-	(junction
 		(at 187.96 90.17)
 		(diameter 0)
@@
 	)
 	(junction
-		(at 176.53 38.1)
-		(diameter 0)
-		(color 0 0 0 0)
-	)
-	(junction
 		(at 66.04 53.34)
 		(diameter 0)
@@
 	)
 	(junction
+		(at 68.58 48.26)
+		(diameter 0)
+		(color 0 0 0 0)
+	)
+	(junction
 		(at 185.42 38.1)
 		(diameter 0)
@@
 	(wire
 		(pts
-			(xy 66.04 48.26) (xy 69.85 48.26)
+			(xy 66.04 48.26) (xy 68.58 48.26)
 		)
 		(stroke
@@
 	(wire
 		(pts
+			(xy 68.58 48.26) (xy 68.58 50.8)
+		)
+		(stroke
+			(width 0)
+			(type default)
+		)
+	)
+	(wire
+		(pts
 			(xy 220.98 95.25) (xy 224.79 95.25)
 		)
@@
 	(wire
 		(pts
+			(xy 68.58 48.26) (xy 69.85 48.26)
+		)
+		(stroke
+			(width 0)
+			(type default)
+		)
+	)
+	(wire
+		(pts
 			(xy 118.11 40.64) (xy 120.65 40.64)
 		)
@@
 	(wire
 		(pts
-			(xy 68.58 43.18) (xy 68.58 50.8)
+			(xy 68.58 43.18) (xy 68.58 48.26)
 		)
 		(stroke
@@
 	(wire
 		(pts
-			(xy 176.53 38.1) (xy 176.53 40.64)
+			(xy 68.58 50.8) (xy 69.85 50.8)
 		)
 		(stroke
@@
 	(wire
 		(pts
-			(xy 68.58 50.8) (xy 69.85 50.8)
-		)
-		(stroke
-			(width 0)
-			(type default)
-		)
-	)
-	(wire
-		(pts
 			(xy 139.7 91.44) (xy 139.7 109.22)
 		)
@@
 			)
 		)
-		(property "Value" "2.2k"
+		(property "Value" "2.7k"
 			(at 184.15 83.82 90)
 			(effects
@@
 		(dnp no)
 		(property "Reference" "C13"
-			(at 50.292 50.038 0)
+			(at 53.086 52.578 0)
 			(effects
 				(font
@@
 		)
 		(property "Value" "10uF"
-			(at 49.53 51.816 0)
+			(at 52.324 53.848 0)
 			(effects
 				(font
@@
 			)
 		)
-		(property "Value" "2.2k"
+		(property "Value" "2.7k"
 			(at 187.96 83.82 90)
 			(effects
@@
 	(symbol
 		(lib_id "power:GND")
-		(at 52.07 48.26 180)
+		(at 52.07 48.26 0)
 		(unit 1)
 		(exclude_from_sim no)
@@
 		(on_board yes)
 		(dnp no)
-		(fields_autoplaced yes)
 		(property "Reference" "#PWR017"
-			(at 52.07 41.91 0)
+			(at 52.07 54.61 0)
 			(effects
 				(font
@@
 		)
 		(property "Value" "GND"
-			(at 52.07 43.18 0)
+			(at 48.26 48.26 0)
 			(effects
 				(font
 					(size 0.889 0.889)
 				)
+				(justify left)
 			)
 		)

Commit message: update
Connections:
- net +3.3V: now also C11.1, C12.2, C13.2, U2.1 (VDDI/O), U2.6 (VS)
- net BMI088_GYRO_INT: no longer U6.13 (INT4)
- no-connect marks 11 -> 12
Other:
- moved on the sheet: C11, C12
Changed lines of the file:
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@@
 	)
 	(junction
-		(at 55.88 48.26)
+		(at 58.42 48.26)
 		(diameter 0)
 		(color 0 0 0 0)
 	)
 	(junction
-		(at 63.5 48.26)
+		(at 55.88 48.26)
 		(diameter 0)
 		(color 0 0 0 0)
@@
 	)
 	(junction
-		(at 66.04 53.34)
+		(at 62.23 53.34)
 		(diameter 0)
 		(color 0 0 0 0)
 	)
 	(junction
-		(at 110.49 92.71)
+		(at 67.31 40.64)
 		(diameter 0)
 		(color 0 0 0 0)
 	)
 	(junction
-		(at 66.04 48.26)
+		(at 67.31 53.34)
 		(diameter 0)
 		(color 0 0 0 0)
@@
 		(color 0 0 0 0)
 	)
+	(junction
+		(at 62.23 48.26)
+		(diameter 0)
+		(color 0 0 0 0)
+	)
 	(no_connect
 		(at 187.96 48.26)
@@
 	)
 	(no_connect
+		(at 109.22 90.17)
+	)
+	(no_connect
 		(at 233.68 43.18)
 	)
@@
 	(wire
 		(pts
-			(xy 66.04 48.26) (xy 68.58 48.26)
+			(xy 110.49 95.25) (xy 114.3 95.25)
 		)
 		(stroke
@@
 	(wire
 		(pts
-			(xy 110.49 95.25) (xy 114.3 95.25)
+			(xy 67.31 40.64) (xy 67.31 53.34)
 		)
 		(stroke
@@
 	(wire
 		(pts
-			(xy 63.5 46.99) (xy 63.5 48.26)
+			(xy 58.42 46.99) (xy 58.42 48.26)
 		)
 		(stroke
@@
 	(wire
 		(pts
-			(xy 142.24 111.76) (xy 148.59 111.76)
+			(xy 67.31 53.34) (xy 69.85 53.34)
 		)
 		(stroke
@@
 	(wire
 		(pts
-			(xy 66.04 53.34) (xy 69.85 53.34)
+			(xy 142.24 111.76) (xy 148.59 111.76)
 		)
 		(stroke
@@
 	(wire
 		(pts
-			(xy 63.5 48.26) (xy 66.04 48.26)
-		)
-		(stroke
-			(width 0)
-			(type default)
-		)
-	)
-	(wire
-		(pts
-			(xy 69.85 40.64) (xy 63.5 40.64)
+			(xy 69.85 40.64) (xy 67.31 40.64)
 		)
 		(stroke
@@
 	(wire
 		(pts
-			(xy 55.88 48.26) (xy 63.5 48.26)
+			(xy 55.88 48.26) (xy 58.42 48.26)
 		)
 		(stroke
@@
 	(wire
 		(pts
-			(xy 63.5 40.64) (xy 63.5 41.91)
+			(xy 58.42 40.64) (xy 58.42 41.91)
 		)
 		(stroke
@@
 	(wire
 		(pts
+			(xy 67.31 38.1) (xy 67.31 40.64)
+		)
+		(stroke
+			(width 0)
+			(type default)
+		)
+	)
+	(wire
+		(pts
 			(xy 184.15 78.74) (xy 184.15 80.01)
 		)
@@
 	(wire
 		(pts
-			(xy 110.49 90.17) (xy 109.22 90.17)
+			(xy 68.58 50.8) (xy 69.85 50.8)
 		)
 		(stroke
@@
 	(wire
 		(pts
-			(xy 68.58 50.8) (xy 69.85 50.8)
+			(xy 144.78 82.55) (xy 144.78 87.63)
 		)
 		(stroke
@@
 	(wire
 		(pts
-			(xy 144.78 82.55) (xy 144.78 87.63)
+			(xy 207.01 114.3) (xy 207.01 116.84)
 		)
 		(stroke
@@
 	(wire
 		(pts
-			(xy 207.01 114.3) (xy 207.01 116.84)
+			(xy 55.88 53.34) (xy 62.23 53.34)
 		)
 		(stroke
@@
 	(wire
 		(pts
-			(xy 55.88 53.34) (xy 66.04 53.34)
+			(xy 109.22 85.09) (xy 111.76 85.09)
 		)
 		(stroke
@@
 	(wire
 		(pts
-			(xy 110.49 90.17) (xy 110.49 92.71)
+			(xy 58.42 92.71) (xy 62.23 92.71)
 		)
 		(stroke
@@
 	(wire
 		(pts
-			(xy 109.22 85.09) (xy 111.76 85.09)
+			(xy 134.62 95.25) (xy 134.62 113.03)
 		)
 		(stroke
@@
 	(wire
 		(pts
-			(xy 58.42 92.71) (xy 62.23 92.71)
+			(xy 69.85 43.18) (xy 68.58 43.18)
 		)
 		(stroke
@@
 	(wire
 		(pts
-			(xy 134.62 95.25) (xy 134.62 113.03)
+			(xy 233.68 53.34) (xy 234.95 53.34)
 		)
 		(stroke
@@
 	(wire
 		(pts
-			(xy 69.85 43.18) (xy 68.58 43.18)
+			(xy 185.42 38.1) (xy 187.96 38.1)
 		)
 		(stroke
@@
 	(wire
 		(pts
-			(xy 233.68 53.34) (xy 234.95 53.34)
+			(xy 109.22 100.33) (xy 113.03 100.33)
 		)
 		(stroke
@@
 	(wire
 		(pts
-			(xy 185.42 38.1) (xy 187.96 38.1)
+			(xy 184.15 85.09) (xy 184.15 87.63)
 		)
 		(stroke
@@
 	(wire
 		(pts
-			(xy 109.22 100.33) (xy 113.03 100.33)
+			(xy 58.42 48.26) (xy 62.23 48.26)
 		)
 		(stroke
@@
 	(wire
 		(pts
-			(xy 184.15 85.09) (xy 184.15 87.63)
+			(xy 62.23 48.26) (xy 68.58 48.26)
 		)
 		(stroke
@@
 	(wire
 		(pts
-			(xy 110.49 92.71) (xy 109.22 92.71)
+			(xy 109.22 92.71) (xy 113.03 92.71)
 		)
 		(stroke
@@
 	(wire
 		(pts
-			(xy 220.98 90.17) (xy 220.98 92.71)
+			(xy 62.23 53.34) (xy 67.31 53.34)
 		)
 		(stroke
@@
 	(wire
 		(pts
-			(xy 118.11 53.34) (xy 120.65 53.34)
+			(xy 220.98 90.17) (xy 220.98 92.71)
 		)
 		(stroke
@@
 	(wire
 		(pts
-			(xy 52.07 48.26) (xy 55.88 48.26)
+			(xy 118.11 53.34) (xy 120.65 53.34)
 		)
 		(stroke
@@
 	(wire
 		(pts
-			(xy 62.23 92.71) (xy 62.23 97.79)
+			(xy 52.07 48.26) (xy 55.88 48.26)
 		)
 		(stroke
@@
 	(wire
 		(pts
-			(xy 110.49 92.71) (xy 113.03 92.71)
+			(xy 62.23 92.71) (xy 62.23 97.79)
 		)
 		(stroke
@@
 	(wire
 		(pts
+			(xy 67.31 40.64) (xy 58.42 40.64)
+		)
+		(stroke
+			(width 0)
+			(type default)
+		)
+	)
+	(wire
+		(pts
 			(xy 144.78 87.63) (xy 144.78 105.41)
 		)
@@
 		(dnp no)
 		(property "Reference" "C13"
-			(at 53.086 52.578 0)
+			(at 52.324 52.324 0)
 			(effects
 				(font
@@
 		)
 		(property "Value" "10uF"
-			(at 52.324 53.848 0)
+			(at 51.816 53.594 0)
 			(effects
 				(font
@@
 	(symbol
 		(lib_id "Device:C_Small")
-		(at 63.5 44.45 0)
+		(at 58.42 44.45 0)
 		(unit 1)
 		(exclude_from_sim no)
@@
 		(dnp no)
 		(property "Reference" "C11"
-			(at 57.15 42.926 0)
+			(at 52.07 42.926 0)
 			(effects
 				(font
@@
 		)
 		(property "Value" "100nF"
-			(at 55.118 44.704 0)
+			(at 50.038 44.704 0)
 			(effects
 				(font
@@
 		)
 		(property "Footprint" "Capacitor_SMD:C_0402_1005Metric"
-			(at 63.5 44.45 0)
+			(at 58.42 44.45 0)
 			(effects
 				(font
@@
 		)
 		(property "Datasheet" "~"
-			(at 63.5 44.45 0)
+			(at 58.42 44.45 0)
 			(effects
 				(font
@@
 		)
 		(property "Description" "Unpolarized capacitor, small symbol"
-			(at 63.5 44.45 0)
+			(at 58.42 44.45 0)
 			(effects
 				(font
@@
 	)
 	(symbol
+		(lib_id "power:+3.3V")
+		(at 67.31 38.1 0)
+		(unit 1)
+		(exclude_from_sim no)
+		(in_bom yes)
+		(on_board yes)
+		(dnp no)
+		(property "Reference" "#PWR0119"
+			(at 67.31 41.91 0)
+			(effects
+				(font
+					(size 1.27 1.27)
+				)
+				(hide yes)
+			)
+		)
+		(property "Value" "+3.3V"
+			(at 67.31 34.036 0)
+			(effects
+				(font
+					(size 1.27 1.27)
+				)
+			)
+		)
+		(property "Footprint" ""
+			(at 67.31 38.1 0)
+			(effects
+				(font
+					(size 1.27 1.27)
+				)
+				(hide yes)
+			)
+		)
+		(property "Datasheet" ""
+			(at 67.31 38.1 0)
+			(effects
+				(font
+					(size 1.27 1.27)
+				)
+				(hide yes)
+			)
+		)
+		(property "Description" "Power symbol creates a global label with name \"+3.3V\""
+			(at 67.31 38.1 0)
+			(effects
+				(font
+					(size 1.27 1.27)
+				)
+				(hide yes)
+			)
+		)
+		(pin "1"
+		)
+		(instances
+			(project ""
+				(path "/f49728bb-5f62-4190-bb7d-54bb4c159a74/cc1d0527-aeda-4a8b-a373-f853681e542f"
+					(reference "#PWR0119")
+					(unit 1)
+				)
+			)
+		)
+	)
+	(symbol
 		(lib_id "EasyEDA:BMI088")
 		(at 87.63 92.71 0)
@@
 	(symbol
 		(lib_id "Device:C_Small")
-		(at 66.04 50.8 0)
+		(at 62.23 50.8 0)
 		(unit 1)
 		(exclude_from_sim no)
@@
 		(dnp no)
 		(property "Reference" "C12"
-			(at 60.452 50.038 0)
+			(at 57.912 50.8 0)
 			(effects
 				(font
@@
 		)
 		(property "Value" "100nF"
-			(at 58.42 51.816 0)
+			(at 57.658 52.324 0)
 			(effects
 				(font
@@
 		)
 		(property "Footprint" "Capacitor_SMD:C_0402_1005Metric"
-			(at 66.04 50.8 0)
+			(at 62.23 50.8 0)
 			(effects
 				(font
@@
 		)
 		(property "Datasheet" "~"
-			(at 66.04 50.8 0)
+			(at 62.23 50.8 0)
 			(effects
 				(font
@@
 		)
 		(property "Description" "Unpolarized capacitor, small symbol"
-			(at 66.04 50.8 0)
+			(at 62.23 50.8 0)
 			(effects
 				(font

Commit message: reroute
Parts:
- R12, R9: value 4.7k -> 2.7k
Connections:
- net BMI088_ACCEL_INT: no longer U6.1 (INT2)
- no-connect marks 12 -> 13
Changed lines of the file:
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@@
 	)
 	(junction
-		(at 64.77 85.09)
-		(diameter 0)
-		(color 0 0 0 0)
-	)
-	(junction
 		(at 111.76 97.79)
 		(diameter 0)
@@
 	)
 	(no_connect
+		(at 66.04 85.09)
+	)
+	(no_connect
 		(at 233.68 48.26)
 	)
@@
 	(wire
 		(pts
-			(xy 64.77 85.09) (xy 64.77 69.85)
-		)
-		(stroke
-			(width 0)
-			(type default)
-		)
-	)
-	(wire
-		(pts
 			(xy 243.84 55.88) (xy 243.84 57.15)
 		)
@@
 	(wire
 		(pts
-			(xy 64.77 85.09) (xy 66.04 85.09)
+			(xy 85.09 69.85) (xy 87.63 69.85)
 		)
 		(stroke
@@
 	(wire
 		(pts
-			(xy 63.5 85.09) (xy 64.77 85.09)
-		)
-		(stroke
-			(width 0)
-			(type default)
-		)
-	)
-	(wire
-		(pts
 			(xy 243.84 35.56) (xy 241.3 35.56)
 		)
@@
 	(wire
 		(pts
-			(xy 64.77 69.85) (xy 87.63 69.85)
-		)
-		(stroke
-			(width 0)
-			(type default)
-		)
-	)
-	(wire
-		(pts
 			(xy 67.31 40.64) (xy 58.42 40.64)
 		)
@@
 	(global_label "BMI088_ACCEL_INT"
 		(shape output)
-		(at 63.5 85.09 180)
+		(at 85.09 69.85 180)
 		(fields_autoplaced yes)
 		(effects
@@
 		)
 		(property "Intersheetrefs" "${INTERSHEET_REFS}"
-			(at 49.0916 85.09 0)
+			(at 70.6816 69.85 0)
 			(effects
 				(font
@@
 			)
 		)
-		(property "Value" "4.7k"
+		(property "Value" "2.7k"
 			(at 240.284 33.782 90)
 			(effects
@@
 			)
 		)
-		(property "Value" "4.7k"
+		(property "Value" "2.7k"
 			(at 181.61 36.322 90)
 			(effects

Commit message: cleanup track and vias
Connections:
- net +3.3V: now also C34.2, U10.2 (VDD)
Changed lines of the file:
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@@
+	)
+	(junction
+		(at 176.53 38.1)
+		(diameter 0)
+		(color 0 0 0 0)
 	)
 	(junction
@@
 	)
 	(junction
+		(at 176.53 40.64)
+		(diameter 0)
+		(color 0 0 0 0)
+	)
+	(junction
 		(at 224.79 87.63)
 		(diameter 0)
@@
 		)
 		(stroke
+			(width 0)
+			(type default)
+		)
+	)
+	(wire
+		(pts
+			(xy 176.53 38.1) (xy 176.53 40.64)
+		)
+		(stroke
