File: FlightCom.kicad_sch (KiCad schematic)
At the start: 50 parts, among them J1 Molex Microfit, J2 Conn_02x03_Counter_Clockwise, U1 TPS62153, U3 LP5912Q3.3DRVRQ1, U4 USBLC6-2SC6, U5 STM32U575VGTx, X1 1XXD32000MBA

Commit message: update
Parts:
- added C47: 100uF, Capacitor_SMD:C_0402_1005Metric_Pad0.74x0.62mm_HandSolder, symbol Device:C_Small
- added H1, H2, H3, H4: MountingHole, MountingHole:MountingHole_2.2mm_M2, symbol Mechanical:MountingHole
- added IC1: SN74HCT125DR, Samacsys:SOIC127P600X175-14N, symbol Samacsys:SN74HCT125DR
- added J10: Conn_01x03_Socket, Connector_Molex:Molex_Micro-Fit_3.0_43650-0315_1x03_P3.00mm_Vertical, symbol Connector:Conn_01x03_Socket
- added J11, J7, J8: Conn_01x02_Socket, Connector_Molex:Molex_Micro-Fit_3.0_43650-0215_1x02_P3.00mm_Vertical, symbol Connector:Conn_01x02_Socket
- added Q1, Q4: SI7232DN-T1-GE3, MOSFET:TRANS_SI7232DN-T1-GE3, symbol MOSFET:SI7232DN-T1-GE3
- added R15, R33, R39: 3.3K, Resistor_SMD:R_0402_1005Metric, symbol Device:R
- added R35, R36, R37, R38: 470R, Resistor_SMD:R_0402_1005Metric_Pad0.72x0.64mm_HandSolder, symbol Device:R_Small
Connections:
- net +5V: now also C47.1, IC1.14 (VCC), J10.3 (Pin_3)
- net GND: now also C47.2, IC1.7 (GND), J10.2 (Pin_2), Q1.1, Q4.1, Q4.3, R15.1, R33.1, R35.2, R36.2, R37.2, R38.2, R39.1
- net GNSS_SafeBoot: no longer U5.81 (PD0)
- net PWM_A: now also IC1.2 (1A)
- net PWM_B: now also IC1.4 (2~{OE})
- net SX1262_BUSY: now also U5.97 (PE0); no longer U5.86 (PD5)
- net SX1262_DIO1: now also U5.98 (PE1); no longer U5.82 (PD1)
- net SX1262_DIO2: now also U5.87 (PD6); no longer U5.88 (PD7)
- net SX1262_DIO3: now also U5.88 (PD7); no longer U5.84 (PD3)
- net SX1262_MOSI: no longer U5.87 (PD6)
- net SX1262_RST: now also U5.93 (PB7); no longer U5.85 (PD4)
- net VBAT+: now also J11.2 (Pin_2), J7.2 (Pin_2), J8.2 (Pin_2)
- net PWM_C: now reaches U5.62 (PD15)
- net PWM_C: now also IC1.9 (3A)
- net PWM_D: now reaches U5.69 (PA10)
- net PWM_D: now also IC1.12 (4A)
- new net: J11.1 (Pin_1), Q1.7, Q1.8
- new net: Q1.5, Q1.6
- new net: J8.1 (Pin_1), Q4.5, Q4.6
- new net: J7.1 (Pin_1), Q4.7, Q4.8
- new net PWM_PD: IC1.1 (1~{OE}), IC1.10 (3~{OE}), IC1.13 (4~{OE}), IC1.5 (2A), R35.1, R36.1, R37.1, R38.1
- new net PYRO_A: IC1.3 (1Y), Q4.2, R39.2
- new net PYRO_B: IC1.6 (2Y), Q4.4, R15.2
- new net PYRO_C: IC1.8 (3Y), Q1.2, R33.2
- new net SERVO_A: IC1.11 (4Y), J10.1 (Pin_1)
- no-connect marks 3 -> 6
Other:
- note added: "Level Shifting"

Commit message: update
Parts:
- H1, H2, H3, H4: footprint MountingHole:MountingHole_2.2mm_M2 -> MountingHole:MountingHole_3.2mm_M3
Changed lines of the file:
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@@
 			)
 		)
-		(property "Footprint" "MountingHole:MountingHole_2.2mm_M2"
+		(property "Footprint" "MountingHole:MountingHole_3.2mm_M3"
 			(at 184.15 41.91 0)
 			(effects
@@
 			)
 		)
-		(property "Footprint" "MountingHole:MountingHole_2.2mm_M2"
+		(property "Footprint" "MountingHole:MountingHole_3.2mm_M3"
 			(at 184.15 46.99 0)
 			(effects
@@
 			)
 		)
-		(property "Footprint" "MountingHole:MountingHole_2.2mm_M2"
+		(property "Footprint" "MountingHole:MountingHole_3.2mm_M3"
 			(at 184.15 31.75 0)
 			(effects
@@
 			)
 		)
-		(property "Footprint" "MountingHole:MountingHole_2.2mm_M2"
+		(property "Footprint" "MountingHole:MountingHole_3.2mm_M3"
 			(at 184.15 36.83 0)
 			(effects

Commit message: reroute
Parts:
- removed C24, C25: 10uF, Capacitor_SMD:C_0402_1005Metric_Pad0.74x0.62mm_HandSolder, symbol Device:C_Small
- removed C3: 100nF, Capacitor_SMD:C_0402_1005Metric_Pad0.74x0.62mm_HandSolder, symbol Device:C_Small
- removed C4: 10pF, Capacitor_SMD:C_0402_1005Metric_Pad0.74x0.62mm_HandSolder, symbol Device:C_Small
- removed D2: MMSZ4683T1G, EasyEDA:SOD-123_L2.8-W1.8-LS3.7-RD, symbol EasyEDA:MMSZ4683T1G
- removed R3: 100k, Resistor_SMD:R_0402_1005Metric_Pad0.72x0.64mm_HandSolder, symbol Device:R_Small
- removed USB1: C169130, EasyEDA:USB-C-SMD_TYPE-C3.1-02, symbol EasyEDA:C169130
- removed X1: 1XXD32000MBA, EasyEDA:OSC-SMD_4P-L2.0-W1.6-BL_1XXD, symbol EasyEDA:1XXD32000MBA
- added D2: MMSZ4683T1G, zener_diode:SOD3716X135N, symbol SamacSys:MMSZ4683T1G
- added USB1: 10172013-00011LF, USBC:AMPHENOL_10172013-00011LF, symbol SamacSys:10172013-00011LF
- added X2: ECS-TXO-32CSMV-320-AN-TR, CLOCK:OSC_ECS-TXO-2520-33-320-AN-TR, symbol SamacSys:ECS-TXO-32CSMV-320-AN-TR
- C21: value 1nF -> 10uF
- C23: value 10uF -> 10nF
Connections:
- net +3.3V: now also X2.4 (VDD)
- net BAT_LEVEL: now also D2.A
- net BCD: now also U5.39 (PE8)
- net D+: now also USB1.A6 (DP1), USB1.B6 (DP2)
- net D-: now also USB1.A7 (DN1), USB1.B7 (DN2)
- net GND: now also C21.1, R5.1, D2.C, USB1.1 (MH1), USB1.2 (MH2), USB1.3 (MH3), USB1.4 (MH4), USB1.A1 (GND_1), USB1.A12 (GND_2), X2.1 (GROUND_1), X2.2 (GROUND_2); no longer C21.2, C23.2, R5.2
- net HSE_IN: now also C23.1
- net VBUS: now also C21.2, USB1.A4 (VBUS_1), USB1.A9 (VBUS_2); no longer C23.1
- net at J11.1 (Pin_1), Q1.7, Q1.8: now also Q1.9
- net at R6.1: now also USB1.B5 (CC2)
- net at J8.1 (Pin_1), Q4.5, Q4.6: now also Q4.10
- net at J7.1 (Pin_1), Q4.7, Q4.8: now also Q4.9
- new net: R5.2, USB1.A5 (CC1)
- new net: C23.2, X2.3 (OUTPUT)
- no-connect marks 6 -> 28
Other:
- note removed: "2 pad only for 4 VBUS"
- moved on the sheet: H1, H2, H3, H4, J2

Commit message: drc checked
Connections:
- net at Q1.5, Q1.6: now also Q1.10
- no-connect marks 28 -> 27
Changed lines of the file:
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@@
 	)
 	(junction
+		(at 134.62 142.24)
+		(diameter 0)
+		(color 0 0 0 0)
+	)
+	(junction
 		(at 254 19.05)
 		(diameter 0)
@@
 	)
 	(no_connect
-		(at 134.62 142.24)
-	)
-	(no_connect
 		(at 269.24 72.39)
 	)
@@
 	(wire
 		(pts
+			(xy 134.62 142.24) (xy 137.16 142.24)
+		)
+		(stroke
+			(width 0)
+			(type default)
+		)
+	)
+	(wire
+		(pts
 			(xy 62.23 138.43) (xy 60.96 138.43)
 		)
@@
 	(wire
 		(pts
+			(xy 137.16 142.24) (xy 137.16 144.78)
+		)
+		(stroke
+			(width 0)
+			(type default)
+		)
+	)
+	(wire
+		(pts
 			(xy 46.99 106.68) (xy 46.99 102.87)
 		)
@@
 	(wire
 		(pts
+			(xy 132.08 144.78) (xy 132.08 142.24)
+		)
+		(stroke
+			(width 0)
+			(type default)
+		)
+	)
+	(wire
+		(pts
 			(xy 73.66 101.6) (xy 71.12 101.6)
 		)
@@
 	(wire
 		(pts
+			(xy 132.08 142.24) (xy 134.62 142.24)
+		)
+		(stroke
+			(width 0)
+			(type default)
+		)
+	)
+	(wire
+		(pts
 			(xy 168.275 62.23) (xy 175.26 62.23)
 		)
@@
 		(pin "9"
 		)
+		(pin "10"
+		)
 		(instances

Commit message: update connection
Connections:
- net BAT_LEVEL: now also U5.35 (PB0)
- no-connect marks 27 -> 26
Changed lines of the file:
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@@
 	)
 	(no_connect
-		(at 269.24 69.85)
-	)
-	(no_connect
 		(at 223.52 57.15)
 	)
@@
 				(hide yes)
 			)
+		)
+	)
+	(global_label "BAT_LEVEL"
+		(shape input)
+		(at 269.24 69.85 0)
+		(fields_autoplaced yes)
+		(effects
+			(font
+				(size 0.889 0.889)
+			)
+			(justify left)
+		)
+		(property "Intersheetrefs" "${INTERSHEET_REFS}"
+			(at 278.1451 69.85 0)
+			(effects
+				(font
+					(size 1.27 1.27)
+				)
+				(justify left)
+				(hide yes)
+			)

Commit message: add buzzer
Parts:
- added LS1: PS1440P02BT, PS1440P02BT:BUZZER_PS1440P02BT, symbol Buzzer:PS1440P02BT
Connections:
- net GND: now also LS1.2
- net PWM_Buzzer: now reaches U5.2 (PE3)
- net PWM_Buzzer: now also LS1.1
- no-connect marks 26 -> 25

Commit message: adjust position
Parts:
- LS1: footprint PS1440P02BT:BUZZER_PS1440P02BT -> Buzzer:BUZZER_PS1440P02BT
Changed lines of the file:
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@@
 			)
 		)
-		(property "Footprint" "PS1440P02BT:BUZZER_PS1440P02BT"
+		(property "Footprint" "Buzzer:BUZZER_PS1440P02BT"
 			(at 166.37 146.05 0)
 			(effects

Commit message: improve routing
Parts:
- H1, H2, H3, H4: footprint MountingHole:MountingHole_3.2mm_M3 -> MountingHole:MountingHole_3.2mm_M3_DIN965_Pad
Connections:
- net VREF+ is gone; now on net +3.3VA: C6.1, U5.21 (VREF+)
Changed lines of the file:
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@@
 	)
 	(junction
+		(at 19.05 123.19)
+		(diameter 0)
+		(color 0 0 0 0)
+	)
+	(junction
 		(at 149.86 111.76)
 		(diameter 0)
@@
 	)
 	(junction
+		(at 27.94 123.19)
+		(diameter 0)
+		(color 0 0 0 0)
+	)
+	(junction
 		(at 96.52 24.13)
 		(diameter 0)
@@
 	(wire
 		(pts
-			(xy 27.94 121.92) (xy 39.37 121.92)
+			(xy 27.94 123.19) (xy 39.37 123.19)
 		)
 		(stroke
@@
 	(wire
 		(pts
+			(xy 19.05 123.19) (xy 27.94 123.19)
+		)
+		(stroke
+			(width 0)
+			(type default)
+		)
+	)
+	(wire
+		(pts
 			(xy 139.7 185.42) (xy 138.43 185.42)
 		)
@@
 		)
 	)
-	(wire
-		(pts
-			(xy 27.94 121.92) (xy 27.94 123.19)
-		)
-		(stroke
-			(width 0)
-			(type default)
-		)
-	)
 	(rectangle
 		(start 68.58 87.63)
@@
 	(global_label "VREF+"
 		(shape passive)
-		(at 39.37 121.92 0)
+		(at 39.37 123.19 0)
 		(fields_autoplaced yes)
 		(effects
@@
 		)
 		(property "Intersheetrefs" "${INTERSHEET_REFS}"
-			(at 47.4125 121.92 0)
+			(at 47.4125 123.19 0)
 			(effects
 				(font
@@
 			)
 		)
-		(property "Footprint" "MountingHole:MountingHole_3.2mm_M3"
+		(property "Footprint" "MountingHole:MountingHole_3.2mm_M3_DIN965_Pad"
 			(at 193.04 41.91 0)
 			(effects
@@
 			)
 		)
-		(property "Footprint" "MountingHole:MountingHole_3.2mm_M3"
+		(property "Footprint" "MountingHole:MountingHole_3.2mm_M3_DIN965_Pad"
 			(at 193.04 46.99 0)
 			(effects
@@
 			)
 		)
-		(property "Footprint" "MountingHole:MountingHole_3.2mm_M3"
+		(property "Footprint" "MountingHole:MountingHole_3.2mm_M3_DIN965_Pad"
 			(at 193.04 31.75 0)
 			(effects
@@
 			)
 		)
-		(property "Footprint" "MountingHole:MountingHole_3.2mm_M3"
+		(property "Footprint" "MountingHole:MountingHole_3.2mm_M3_DIN965_Pad"
 			(at 193.04 36.83 0)
 			(effects
