File: FlightCom.kicad_sch (KiCad schematic)
At the start: 65 parts, among them IC1 SN74HCT125DR, J1 Molex Microfit, J10 Conn_01x03_Socket, J11 Conn_01x02_Socket, J2 Conn_02x03_Counter_Clockwise, J7 Conn_01x02_Socket, J8 Conn_01x02_Socket, Q1 SI7232DN-T1-GE3, Q4 SI7232DN-T1-GE3, U1 TPS62153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

Commit message: improve
Parts:
- removed J2: Conn_02x03_Counter_Clockwise, Connector_PinHeader_2.54mm:PinHeader_2x03_P2.54mm_Vertical, symbol Connector_Generic:Conn_02x03_Counter_Clockwise
- added C16, C24: 100uF, Capacitor_SMD:C_0402_1005Metric_Pad0.74x0.62mm_HandSolder, symbol Device:C_Small
- added C25: 10uF, Capacitor_SMD:C_0402_1005Metric_Pad0.74x0.62mm_HandSolder, symbol Device:C_Small
- added J4: Conn_02x04_Counter_Clockwise, Connector_PinHeader_2.54mm:PinHeader_2x04_P2.54mm_Vertical, symbol Connector_Generic:Conn_02x04_Counter_Clockwise
- added R16, R18, R23: 5R, Resistor_SMD:R_0402_1005Metric, symbol Device:R
Connections:
- net +3.3V: now also C16.2, J4.8 (Pin_8)
- net BOOT0: now also J4.5 (Pin_5)
- net COMPANION_RX: now also J4.4 (Pin_4)
- net COMPANION_TX: now also J4.6 (Pin_6)
- net GND: now also C16.1, C24.1, C25.1, J4.7 (Pin_7)
- net SWCLK: now also J4.3 (Pin_3)
- net SWDIO: now also J4.2 (Pin_2)
- net VBAT+: now also C24.2, C25.2, R16.1, R18.1, R23.1; no longer J11.2 (Pin_2), J7.2 (Pin_2), J8.2 (Pin_2)
- net nRST: now also J4.1 (Pin_1)
- new net: J11.2 (Pin_2), R23.2
- new net: J8.2 (Pin_2), R18.2
- new net: J7.2 (Pin_2), R16.2
Other:
- moved on the sheet: D1, D9, J1, J8, R22

Commit message: for frab
Changed lines of the file:
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@@
 	(rectangle
 		(start 114.3 87.63)
-		(end 179.07 128.27)
+		(end 185.42 128.27)
 		(stroke
 			(width 0)

Commit message: updated schematic
Parts:
- removed J11: Conn_01x02_Socket, Connector_Molex:Molex_Micro-Fit_3.0_43650-0215_1x02_P3.00mm_Vertical, symbol Connector:Conn_01x02_Socket
- removed Q1: SI7232DN-T1-GE3, MOSFET:TRANS_SI7232DN-T1-GE3, symbol MOSFET:SI7232DN-T1-GE3
- removed R23: 5R, Resistor_SMD:R_0402_1005Metric, symbol Device:R
- removed R33: 3.3K, Resistor_SMD:R_0402_1005Metric, symbol Device:R
- added J2: Conn_01x03_Socket, Connector_Molex:Molex_Micro-Fit_3.0_43650-0315_1x03_P3.00mm_Vertical, symbol Connector:Conn_01x03_Socket
- added R23: 1K, Resistor_SMD:R_0402_1005Metric_Pad0.72x0.64mm_HandSolder, symbol Device:R_Small
- added R24, R25: 5R, Resistor_SMD:R_0402_1005Metric, symbol Device:R
Connections:
- net +5V: now also J2.3 (Pin_3)
- net GND: now also J2.2 (Pin_2)
- net PWM_B: now also IC1.5 (2A); no longer IC1.4 (2~{OE})
- net PWM_Buzzer: now also R23.1; no longer LS1.1
- net PWM_PD: now also IC1.4 (2~{OE}); no longer IC1.5 (2A)
- net SERVO_A: now also R24.1; no longer J10.1 (Pin_1)
- net PYRO_C renamed SERVO_C
- net SERVO_C: now also R25.1
- new net: J10.1 (Pin_1), R24.2
- new net: J2.1 (Pin_1), R25.2
- new net: LS1.1, R23.2
- no-connect marks 25 -> 23
Other:
- moved on the sheet: LS1
