File: FlightCom.kicad_pcb (KiCad board)
At the start: 4 copper layers, 88.4 x 62.4 mm, 147 parts, among them IC1 SN74HCT125DR, J1 Molex Microfit, J10 Conn_01x03_Socket, J11 Conn_01x02_Socket, J3 RF2-04A-T-00-50-G, J4 Conn_02x04_Counter_Clockwise, J7 Conn_01x02_Socket, J8 Conn_01x02_Socket, J9 BMI-S-209-F, Q1 SI7232DN-T1-GE3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

Commit message: for frab
Parts:
- moved LOGO 2.21 mm to (143.2, 87.5)
- moved H4 1.31 mm to (174.0, 110.0)
- moved H2 1.21 mm to (95.0, 57.5)
- moved H3 1.14 mm to (174.0, 57.5)
- moved H1 0.99 mm to (95.0, 110.0)
- moved C1 0.83 mm to (146.0, 91.5)
- moved R22 0.19 mm to (147.0, 93.7)
Routing:
- net +3.3V: track 134.5 -> 134.0 mm
Other:
- board text added: "3.3V"
- board text added: "5V"
- board text added: "BOOT0"
- board text added: "FET"
- board text added: "GND"
- board text added: "NRST"
- board text added: "RX"
- board text added: "SWCLK"
- board text added: "SWDIO"
- board text added: "TX"
- board text added: "VBAT+"

Commit message: updated schematic
Parts:
- removed J11: Conn_01x02_Socket, Connector_Molex:Molex_Micro-Fit_3.0_43650-0215_1x02_P3.00mm_Vertical
- removed Q1: SI7232DN-T1-GE3, MOSFET:TRANS_SI7232DN-T1-GE3
- removed R23: 5R, Resistor_SMD:R_0402_1005Metric
- removed R33: 3.3K, Resistor_SMD:R_0402_1005Metric
- added J2: Conn_01x03_Socket, Connector_Molex:Molex_Micro-Fit_3.0_43650-0315_1x03_P3.00mm_Vertical, F.Cu at (166.2, 56.4)
- moved LOGO 0.90 mm to (102.2, 74.0)
Routing:
- net PYRO_C: track 18.4 -> 40.4 mm
- net VBAT+: track 49.2 -> 27.4 mm
- net Net-(J11-Pin_1): track 19.7 -> 0.00 mm
- net Net-(J11-Pin_2): track 4.35 -> 0.00 mm
- net VBAT-: track 156.7 -> 154.5 mm, vias 113 -> 111
- net BAT_LEVEL: track 48.4 -> 46.4 mm
