File: IREC-FlighComputer.kicad_pcb (KiCad board)
At the start: 4 copper layers, 109 x 59 mm, 146 parts, among them IC1 SN74HCT125DR, J1 Molex Microfit, J10 Conn_01x03_Socket, J2 Conn_01x03_Socket, J3 RF2-04A-T-00-50-G, J4 Conn_02x04_Counter_Clockwise, J5 BMI-S-209-F, J7 Conn_01x02_Socket, J8 Conn_01x02_Socket, Q4 SI7232DN-T1-GE3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

Commit message: update layout
Parts:
- added D10: LED, LED_SMD:LED_0402_1005Metric, F.Cu at (144.8, 80.9)
- added R33: 1k, Resistor_SMD:R_0402_1005Metric, F.Cu at (147.4, 80.9)
Connections:
- U5 pad 1: unconnected-(U5-PE2-Pad1) -> Debug_LED
Routing:
- net Net-(D3-K): track 11.4 -> 16.3 mm
- net Debug_LED: track 0.00 -> 3.59 mm
- net SX1262_SCK: track 25.8 -> 27.6 mm
- net Net-(D10-A): track 0.00 -> 1.63 mm
- net SX1262_MOSI: track 24.8 -> 26.2 mm
- net SX1262_NSS: track 29.8 -> 31.2 mm
- net SX1262_DIO3: track 15.9 -> 17.1 mm
- net SX1262_MISO: track 23.0 -> 23.9 mm
- net VBAT-: vias 90 -> 91
