File: IREC-FlighComputer.kicad_sch (KiCad schematic)
At the start: 71 parts, among them IC1 SN74HCT125DR, J1 Molex Microfit, J10 Conn_01x03_Socket, J2 Conn_01x03_Socket, J4 Conn_02x04_Counter_Clockwise, J7 Conn_01x02_Socket, J8 Conn_01x02_Socket, Q4 SI7232DN-T1-GE3, U1 TPS62153, U3 LP5912Q3.3DRVRQ1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

Commit message: update layout
Parts:
- added D10: LED, LED_SMD:LED_0402_1005Metric, symbol Device:LED
- added R33: 1k, Resistor_SMD:R_0402_1005Metric, symbol Device:R
Connections:
- net GND: now also D10.1 (K)
- net Debug_LED: now reaches U5.1 (PE2)
- net Debug_LED: now also R33.1
- new net: D10.2 (A), R33.2
- no-connect marks 22 -> 21
Other:
- moved on the sheet: J10, J2, R24, R25
